File: src/kicad/DC Electronic Load.kicad_sch (KiCad schematic)
At the start: 0 parts

Commit message: Tidy up kicad schematic
Other:
- sheet DC Electronic Load_1 renamed Load
- sheet DC Electronic Load_3 renamed Power Supplies
- title: (none) -> DC Electronic Load
Changed lines of the file:
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@@
 (kicad_sch (version 20230121) (generator eeschema)
   (paper "A4")
-  (sheet (at 76.2 25.4) (size 12.7 3.81) (fields_autoplaced)
+  (title_block
+    (title "DC Electronic Load")
+    (date "2023-07-13")
+  )
+  (sheet (at 135.89 92.71) (size 12.7 3.81) (fields_autoplaced)
     (stroke (width 0) (type solid))
     (fill (color 0 0 0 0.0000))
-    (property "Sheetname" "DC Electronic Load_2" (at 76.2 24.6884 0)
+    (property "Sheetname" "DC Electronic Load_2" (at 135.89 91.9984 0)
       (effects (font (size 1.27 1.27)) (justify left bottom))
     )
-    (property "Sheetfile" "DC_Electronic_Load_2.kicad_sch" (at 76.2 29.7946 0)
+    (property "Sheetfile" "DC_Electronic_Load_2.kicad_sch" (at 135.89 97.1046 0)
       (effects (font (size 1.27 1.27)) (justify left top))
     )
@@
     )
   )
-  (sheet (at 127 25.4) (size 12.7 3.81) (fields_autoplaced)
+  (sheet (at 186.69 92.71) (size 12.7 3.81) (fields_autoplaced)
     (stroke (width 0) (type solid))
     (fill (color 0 0 0 0.0000))
-    (property "Sheetname" "DC Electronic Load_3" (at 127 24.6884 0)
+    (property "Sheetname" "Power Supplies" (at 186.69 91.9984 0)
       (effects (font (size 1.27 1.27)) (justify left bottom))
     )
-    (property "Sheetfile" "DC_Electronic_Load_3.kicad_sch" (at 127 29.7946 0)
+    (property "Sheetfile" "DC_Electronic_Load_3.kicad_sch" (at 186.69 97.1046 0)
       (effects (font (size 1.27 1.27)) (justify left top))
     )
@@
     )
   )
-  (sheet (at 25.4 25.4) (size 12.7 3.81) (fields_autoplaced)
+  (sheet (at 85.09 92.71) (size 12.7 3.81) (fields_autoplaced)
     (stroke (width 0) (type solid))
     (fill (color 0 0 0 0.0000))
-    (property "Sheetname" "DC Electronic Load_1" (at 25.4 24.6884 0)
+    (property "Sheetname" "Load" (at 85.09 91.9984 0)
       (effects (font (size 1.27 1.27)) (justify left bottom))
     )
-    (property "Sheetfile" "DC_Electronic_Load_1.kicad_sch" (at 25.4 29.7946 0)
+    (property "Sheetfile" "DC_Electronic_Load_1.kicad_sch" (at 85.09 97.1046 0)
       (effects (font (size 1.27 1.27)) (justify left top))
     )
