File: src/kicad/DC_Electronic_Load_1.kicad_sch (KiCad schematic)
At the start: 60 parts, among them K1 AZ8-FORM-C, Q1 IRFP240, Q10 IRFP240, Q11 NPN, Q12 IRFP240, Q13 IRFP240, Q14 IRFP240, Q15 IRFP240, Q2 IRFP240, Q3 IRFP240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

Commit message: Tidy up kicad schematic
Other:
- title: (none) -> DC Electronic Load
- moved on the sheet: C1, C10, C11, C12, C13, C14, C15, C2, C3, Q1, Q10, Q11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
