File: src/kicad/DC_Electronic_Load_2.kicad_sch (KiCad schematic)
At the start: 23 parts, among them IC1 LM393D, IC2 TL072D, K1 AZ8-FORM-C, Q9 NPN, U4 SN74AHC08

Commit message: Tidy up kicad schematic
Other:
- title: (none) -> DC Electronic Load
- moved on the sheet: D3, Q9, R20, R21, R22, R23, R24, R25, R26, R27, R28, R29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
